File: hardware/kicad/ESPKey.kicad_pcb (KiCad board)
At the start: 2 copper layers, 16 x 20 mm, 32 parts, among them P1 Power, P2 Wiegand, Q1 2N7002, Q2 2N7002, Q3 2N7002, U1 RT6212A/B, U2 ESP-12

Commit message: Open KiCad design in current version of KiCad and remap symbols
Other:
- net class Default removed
